File: rtcc_boosterpack.kicad_sch (KiCad schematic)
At the start: 19 parts, among them J1 TI_BOOSTER_40_J1, J2 TI_BOOSTER_40_J2, J3 TI_BOOSTER_40_J3, J4 TI_BOOSTER_40_J4, J5 Micro_SD_Card_Det, J6 Screw_Terminal_01x04, J7 Screw_Terminal_01x02, M1 DS3234, U1 TB6612FNG

Commit message: Fixes D1 polarity.
Connections:
- net +3V3: now also D1.2 (A); no longer D1.1 (K)
- net at R2.1: now also D1.1 (K); no longer D1.2 (A)
Other:
- moved on the sheet: D1

Commit message: Updates revision number in design sheet.
Other:
- title: (none) -> RTCC BoosterPack
Changed lines of the file:
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@@
   (paper "A4")
   (title_block
+    (title "RTCC BoosterPack")
     (date "19 oct 2012")
+    (rev "1.1")
   )
   (junction (at 66.04 92.71) (diameter 0) (color 0 0 0 0)
