File: rtcc_boosterpack.kicad_pcb (KiCad board)
At the start: 2 copper layers, 50.8 x 38.1 mm, 19 parts, among them J1 TI_BOOSTER_40_J1, J2 TI_BOOSTER_40_J2, J3 TI_BOOSTER_40_J3, J4 TI_BOOSTER_40_J4, J5 Micro_SD_Card_Det, J6 Screw_Terminal_01x04, J7 Screw_Terminal_01x02, M1 DS3234, U1 TB6612FNG

Commit message: Fixes D1 polarity.
Parts:
- C1, C5, C6: value 22uF/10V -> 22uF/25V
- C3: value 22uF/20V -> 22uF/25V
- RN1, RN2: value 47K -> 10K
- turned D1 to 180 degrees
Connections:
- D1 pad 1: +3V3 -> Net-(D1-K)
- D1 pad 2: Net-(D1-Pad2) -> +3V3
- J1 pad 10: Net-(J1-Pad10) -> unconnected-(J1-1.10/PA7-Pad10)
- J1 pad 2: Net-(J1-Pad2) -> unconnected-(J1-1.02/PB5-Pad2)
- J1 pad 3: Net-(J1-Pad3) -> unconnected-(J1-1.03/PB0/Rxd-Pad3)
- J1 pad 4: Net-(J1-Pad4) -> unconnected-(J1-1.04/PB1/TxD-Pad4)
- J1 pad 6: Net-(J1-Pad6) -> unconnected-(J1-1.06/PE5-Pad6)
- J1 pad 8: Net-(J1-Pad8) -> unconnected-(J1-1.08/PA5-Pad8)
- J1 pad 9: Net-(J1-Pad9) -> unconnected-(J1-1.09/PA6-Pad9)
- J2 pad 2: Net-(J2-Pad2) -> unconnected-(J2-2.02/PB2-Pad2)
- J2 pad 3: Net-(J2-Pad3) -> unconnected-(J2-2.03/PE0-Pad3)
- J2 pad 5: Net-(J2-Pad5) -> unconnected-(J2-2.05/RESET-Pad5)
- J3 pad 1: Net-(J3-Pad1) -> unconnected-(J3-3.01/+5V-Pad1)
- J3 pad 10: Net-(J3-Pad10) -> unconnected-(J3-3.10/PF1-Pad10)
- J3 pad 3: Net-(J3-Pad3) -> unconnected-(J3-3.03/PD0-Pad3)
- J3 pad 4: Net-(J3-Pad4) -> unconnected-(J3-3.04/PD1-Pad4)
- J3 pad 5: Net-(J3-Pad5) -> unconnected-(J3-3.05/PD2-Pad5)
- J3 pad 6: Net-(J3-Pad6) -> unconnected-(J3-3.06/PD3-Pad6)
- J3 pad 7: Net-(J3-Pad7) -> unconnected-(J3-3.07/PE1-Pad7)
- J3 pad 8: Net-(J3-Pad8) -> unconnected-(J3-3.08/PE2-Pad8)
- J3 pad 9: Net-(J3-Pad9) -> unconnected-(J3-3.09/PE3-Pad9)
- J4 pad 3: Net-(J4-Pad3) -> unconnected-(J4-4.03/PB3-Pad3)
- J4 pad 4: Net-(J4-Pad4) -> unconnected-(J4-4.04/PC4-Pad4)
- J4 pad 5: Net-(J4-Pad5) -> unconnected-(J4-4.05/PC5-Pad5)
- J5 pad 10: Net-(J5-Pad10) -> unconnected-(J5-DET_A-Pad10)
- M1 pad 3: Net-(M1-Pad3) -> unconnected-(M1-32KHZ-Pad3)
- R2 pad 1: Net-(D1-Pad2) -> Net-(D1-K)
Routing:
- net Net-(D1-Pad2): track 2.90 -> 0.00 mm
- net Net-(D1-K): track 0.00 -> 2.90 mm

Commit message: Updates version printed on bottom silk screen.
Other:
- board text added: "PFPP Booster Pack Martin Garon, Nov 2021 rev 1.1"
- board text removed: "PFPP Booster Pack Martin Garon, Nov 2021 rev 1.0"
Changed lines of the file:
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@@
     (effects (font (size 1 1) (thickness 0.15)) (justify mirror))
   )
-  (gr_text "PFPP Booster Pack\nMartin Garon, Nov 2021\nrev 1.0" (at 193.04 115.062) (layer "B.SilkS")
+  (gr_text "PFPP Booster Pack\nMartin Garon, Nov 2021\nrev 1.1" (at 193.04 115.062) (layer "B.SilkS")
     (effects (font (size 1 1) (thickness 0.15)) (justify mirror))
   )
